File: kicad_pcb/synthesizer/synthesizer.kicad_pcb (KiCad board)
At the start: 2 copper layers, 69.9 x 64.5 mm, 44 parts, among them J1 SCL_GND_SCA, J2 Fuente5V, J3 Fuente5V, J4 Fuente12V, J5 CONSMA006.062-G, Q1 BCW31_

Commit message: Cambio de huella
Parts:
- removed J3: Fuente5V, Connector_PinHeader_2.54mm:PinHeader_1x02_P2.54mm_Vertical
- SP1: footprint Package_SO:SSOP-16_3.9x4.9mm_P0.635mm -> Package_SO:SOP-16_4.55x10.3mm_P1.27mm
- moved C11 5.80 mm to (191.2, 110.3)
- moved C9 1.78 mm to (162.0, 96.0), turned to 0 degrees
- moved SP1 1.17 mm to (163.8, 105.1)
- moved C6 0.93 mm to (170.1, 107.5)
Routing:
- net +5V: track 89.9 -> 116.7 mm, vias 0 -> 4
- net Net-(SP1-Crystal_Cap): track 14.4 -> 11.7 mm
- net Net-(SP1-Charge_Pump): track 4.52 -> 7.13 mm
- net Net-(J1-Pin_3): track 12.8 -> 11.4 mm
- net Net-(SP1-Drive): track 6.38 -> 5.02 mm
- net Net-(SP1-Crystal): track 26.1 -> 25.1 mm
- net Net-(C8-Pad2): track 7.43 -> 8.06 mm
- net Net-(C6-Pad2): track 3.74 -> 4.25 mm
- net GND: vias 76 -> 74
