File: kicad_pcb/synthesizer/synthesizer.kicad_sch (KiCad schematic)
At the start: 44 parts, among them J1 SCL_GND_SCA, J2 Fuente5V, J3 Fuente5V, J4 Fuente12V, J5 CONSMA006.062-G, Q1 BCW31_

Commit message: Cambio de huella
Parts:
- removed J3: Fuente5V, Connector_PinHeader_2.54mm:PinHeader_1x02_P2.54mm_Vertical, symbol Connector:Conn_01x02_Pin
- SP1: footprint Package_SO:SSOP-16_3.9x4.9mm_P0.635mm -> Package_SO:SOP-16_4.55x10.3mm_P1.27mm
Changed lines of the file:
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@@
 	)
 	(junction
-		(at 33.02 114.3)
-		(diameter 0)
-		(color 0 0 0 0)
-	)
-	(junction
 		(at 72.39 82.55)
 		(diameter 0)
@@
 		(color 0 0 0 0)
 	)
-	(junction
-		(at 30.48 124.46)
-		(diameter 0)
-		(color 0 0 0 0)
-	)
 	(no_connect
 		(at 86.36 106.68)
@@
 	(wire
 		(pts
-			(xy 25.4 124.46) (xy 30.48 124.46)
-		)
-		(stroke
-			(width 0)
-			(type default)
-		)
-	)
-	(wire
-		(pts
 			(xy 73.66 34.29) (xy 78.74 34.29)
 		)
@@
 	(wire
 		(pts
-			(xy 30.48 124.46) (xy 30.48 125.73)
+			(xy 30.48 116.84) (xy 30.48 125.73)
 		)
 		(stroke
@@
 	(wire
 		(pts
-			(xy 30.48 116.84) (xy 30.48 124.46)
-		)
-		(stroke
-			(width 0)
-			(type default)
-		)
-	)
-	(wire
-		(pts
 			(xy 168.91 81.28) (xy 173.99 81.28)
 		)
@@
 	(wire
 		(pts
-			(xy 25.4 121.92) (xy 33.02 121.92)
-		)
-		(stroke
-			(width 0)
-			(type default)
-		)
-	)
-	(wire
-		(pts
 			(xy 124.46 71.12) (xy 124.46 69.85)
 		)
@@
 	(wire
 		(pts
-			(xy 33.02 114.3) (xy 35.56 114.3)
-		)
-		(stroke
-			(width 0)
-			(type default)
-		)
-	)
-	(wire
-		(pts
 			(xy 72.39 80.01) (xy 72.39 82.55)
 		)
@@
 	(wire
 		(pts
-			(xy 33.02 121.92) (xy 33.02 114.3)
-		)
-		(stroke
-			(width 0)
-			(type default)
-		)
-	)
-	(wire
-		(pts
 			(xy 184.15 69.85) (xy 184.15 82.55)
 		)
@@
 	(wire
 		(pts
-			(xy 29.21 114.3) (xy 33.02 114.3)
+			(xy 29.21 114.3) (xy 35.56 114.3)
 		)
 		(stroke
@@
 	)
 	(symbol
-		(lib_id "Connector:Conn_01x02_Pin")
-		(at 20.32 121.92 0)
-		(unit 1)
-		(exclude_from_sim no)
-		(in_bom yes)
-		(on_board yes)
-		(dnp no)
-		(property "Reference" "J3"
-			(at 20.32 125.984 0)
-			(effects
-				(font
-					(size 1.27 1.27)
-				)
-			)
-		)
-		(property "Value" "Fuente5V"
-			(at 20.955 119.38 0)
-			(effects
-				(font
-					(size 1.27 1.27)
-				)
-			)
-		)
-		(property "Footprint" "Connector_PinHeader_2.54mm:PinHeader_1x02_P2.54mm_Vertical"
-			(at 20.32 121.92 0)
-			(effects
-				(font
-					(size 1.27 1.27)
-				)
-				(hide yes)
-			)
-		)
-		(property "Datasheet" "~"
-			(at 20.32 121.92 0)
-			(effects
-				(font
-					(size 1.27 1.27)
-				)
-				(hide yes)
-			)
-		)
-		(property "Description" "Generic connector, single row, 01x02, script generated"
-			(at 20.32 121.92 0)
-			(effects
-				(font
-					(size 1.27 1.27)
-				)
-				(hide yes)
-			)
-		)
-		(pin "2"
-		)
-		(pin "1"
-		)
-		(instances
-			(project "synthesizer"
-				(path "/d408f72c-bd6c-4684-9fbd-f8c0676a6c58"
-					(reference "J3")
-					(unit 1)
-				)
-			)
-		)
-	)
-	(symbol
 		(lib_id "BCW31_:BCW31_")
 		(at 121.92 76.2 0)
@@
 			)
 		)
-		(property "Footprint" "Package_SO:SSOP-16_3.9x4.9mm_P0.635mm"
+		(property "Footprint" "Package_SO:SOP-16_4.55x10.3mm_P1.27mm"
 			(at 88.9 85.09 0)
 			(effects
